Commit message: gmapping_wall

File: my_velodyne_description/urdf/VLP-16.urdf.xacro (robot description, xacro)
@@ -2,5 +2,5 @@
 <robot xmlns:xacro="http://www.ros.org/wiki/xacro" name="VLP-16">
   <xacro:property name="M_PI" value="3.1415926535897931" />
-  <xacro:macro name="VLP-16" params="*origin parent:=support name:=velodyne topic:=/velodyne_points organize_cloud:=false hz:=5 lasers:=8 samples:=600 collision_range:=0.3 min_range:=0.9 max_range:=100.0 noise:=0.008 min_angle:=-${M_PI} max_angle:=${M_PI} gpu:=false">
+  <xacro:macro name="VLP-16" params="*origin parent:=support name:=velodyne topic:=/velodyne_points organize_cloud:=false hz:=5 lasers:=8 samples:=1000 collision_range:=0.3 min_range:=0.9 max_range:=100.0 noise:=0.008 min_angle:=-${M_PI} max_angle:=${M_PI} gpu:=false">
     <!-- 支架定义 -->
     <xacro:property name="support_length" value="0.15" /> <!-- 支架长度 -->
